Commit message: added torque sensors

File: src/exoskeleton_description/urdf/exo.xacro (robot description, xacro)
@@ -30,5 +30,4 @@
   <safety_controller k_velocity="20" soft_lower_limit="-0.665" soft_upper_limit="0.665"/> <!-- 0.665rad ~= 38° -->
 </joint>
-<!-- Thigh Link -->
 <link name="thigh_link">
   <visual>
@@ -36,9 +35,20 @@
     <material name="blue"><color rgba="0 0 0.8 1"/></material>
   </visual>
-  <collision><geometry><cylinder length="0.3" radius="0.03"/></geometry></collision>
-  <inertial>
+  <collision>
+    <geometry><cylinder length="0.3" radius="0.03"/></geometry>
+  </collision>
+  <!-- Inertial (Adj. accordingly to the real setup) -->
+  <inertial>
+    <origin xyz="0 0 0.15"/>  <!-- certer of mass in the middle -->
     <mass value="0.5"/>
-    <inertia ixx="0.005" ixy="0" ixz="0" iyy="0.005" iyz="0" izz="0.005"/>
-  </inertial>
+    <inertia ixx="0.00375" ixy="0" ixz="0" iyy="0.00375" iyz="0" izz="0.00045"/>
+  </inertial>
+  <!-- Gazebo Attr -->
+  <gazebo reference="thigh_link">
+    <mu1>0.2</mu1>  <!-- Contact Friction Coefficient -->
+    <mu2>0.2</mu2>
+    <kp>1000000</kp>  <!-- Contact Stiffness [N/m] -->
+    <kd>100</kd>      <!-- Contact Damping [N·s/m] -->
+  </gazebo>
 </link>
 <!-- Knee Joint -->
@@ -71,4 +81,11 @@
     <inertia ixx="0.003" ixy="0" ixz="0" iyy="0.003" iyz="0" izz="0.003"/>
   </inertial>
+  <!-- Gazebo Attr -->
+  <gazebo reference="thigh_link">
+    <mu1>0.2</mu1>  <!-- Contact Friction Coefficient -->
+    <mu2>0.2</mu2>
+    <kp>1000000</kp>  <!-- Contact Stiffness [N/m] -->
+    <kd>100</kd>      <!-- Contact Damping [N·s/m] -->
+  </gazebo>
 </link>
 <!-- Ankle Joint -->
@@ -99,6 +116,13 @@
     <inertia ixx="0.0001" ixy="0" ixz="0" iyy="0.0001" iyz="0" izz="0.0001"/>
   </inertial>
-</link>
-<!-- Transmissions (unchanged) -->
+  <!-- Gazebo Attr -->
+  <gazebo reference="thigh_link">
+    <mu1>0.2</mu1>  <!-- Contact Friction Coefficient -->
+    <mu2>0.2</mu2>
+    <kp>1000000</kp>  <!-- Contact Stiffness [N/m] -->
+    <kd>100</kd>      <!-- Contact Damping [N·s/m] -->
+  </gazebo>
+</link>
+<!-- Transmissions -->
 <transmission name="hip_transmission">
   <type>transmission_interface/SimpleTransmission</type>
@@ -122,5 +146,6 @@
   <joint name="ankle_joint"/>
 </transmission>
-<!-- Gazebo plugins (unchanged) -->
+<!-- Gazebo plugins -->
+<!-- IMU -->
 <gazebo reference="thigh_link">
   <sensor type="imu" name="thigh_imu">
@@ -129,14 +154,70 @@
   </sensor>
 </gazebo>
+<!-- Force Torque Sensors -->
+<gazebo reference="thigh_link">
+  <sensor name="hip_torque_sensor" type="force_torque">
+    <update_rate>100</update_rate>
+    <plugin filename="libgazebo_ros_ft_sensor.so" name="ft_sensor_plugin">
+      <topic>hip_joint_torque</topic>
+      <update_rate>100</update_rate>
+    </plugin>
+    <force_torque>
+      <frame>child</frame>
+      <measure_direction>child_to_parent</measure_direction>
+    </force_torque>
+    <noise>
+      <type>gaussian</type>
+      <mean>0</mean>
+      <stddev>0.02</stddev>  <!-- 2% std noise -->
+    </noise>
+  </sensor>
+</gazebo>
+<gazebo reference="shank_link">
+  <sensor name="knee_torque_sensor" type="force_torque">
+    <update_rate>100</update_rate>
+    <plugin filename="libgazebo_ros_ft_sensor.so" name="ft_sensor_plugin">
+      <topic>knee_joint_torque</topic>
+      <update_rate>100</update_rate>
+    </plugin>
+    <force_torque>
+      <frame>child</frame>
+      <measure_direction>child_to_parent</measure_direction>
+    </force_torque>
+    <noise>
+      <type>gaussian</type>
+      <mean>0</mean>
+      <stddev>0.02</stddev>  <!-- 2% std noise -->
+    </noise>
+  </sensor>
+</gazebo>
 <gazebo reference="foot_link">
-  <sensor type="contact" name="foot_contact">
-    <always_on>true</always_on>
-    <update_rate>50</update_rate>
-  </sensor>
-</gazebo>
-<gazebo>
-  <plugin name="gazebo_ros_control" filename="libgazebo_ros_control.so">
-    <robotNamespace>/exoskeleton</robotNamespace>
-  </plugin>
-</gazebo>
+  <sensor name="ankle_torque_sensor" type="force_torque">
+    <update_rate>100</update_rate>
+    <plugin filename="libgazebo_ros_ft_sensor.so" name="ft_sensor_plugin">
+      <topic>ankle_joint_torque</topic>
+      <update_rate>100</update_rate>
+    </plugin>
+    <force_torque>
+      <frame>child</frame>
+      <measure_direction>child_to_parent</measure_direction>
+    </force_torque>
+    <noise>
+      <type>gaussian</type>
+      <mean>0</mean>
+      <stddev>0.02</stddev>  <!-- 2% std noise -->
+    </noise>
+  </sensor>
+</gazebo>
+  <!-- Contact Sensor -->
+  <gazebo reference="foot_link">
+    <sensor type="contact" name="foot_contact">
+      <always_on>true</always_on>
+      <update_rate>50</update_rate>
+    </sensor>
+  </gazebo>
+  <gazebo>
+    <plugin name="gazebo_ros_control" filename="libgazebo_ros_control.so">
+      <robotNamespace>/exoskeleton</robotNamespace>
+    </plugin>
+  </gazebo>
 </robot>
