Commit message: fixed bugs in URDF

File: src/exo_urdf/urdf/exo.urdf (robot description, URDF)
Before this commit: robot exoskeleton_leg, 4 links, 3 joints
Links:
- link shank_link: mass 0.3 -> 0.25
Joints:
- joint ankle_joint: limit lower=-0.3 upper=0.3 effort=300 velocity=3.0 -> lower=-0.3 upper=0.3 effort=150 velocity=3.0

File: src/exo_urdf/urdf/exo.xacro (robot description, xacro)
@@ -1,11 +1,98 @@
 <?xml version="1.0"?>
-<robot name="exoskeleton_leg" xmlns:xacro="http://ros.org/wiki/xacro">
+<robot name="exo_leg" xmlns:xacro="http://ros.org/wiki/xacro">
   <!-- Properties -->
   <xacro:property name="motor_mass" value="3" />  <!-- Hip / Knee motor mass (kg) -->
   <xacro:property name="base_mass" value="1.0" />   <!-- Base structure mass -->
+  <!-- IMU Sensor Macro -->
+  <xacro:macro name="imu_sensor" params="link_reference sensor_name topic_suffix update_rate:=100">
+    <gazebo reference="${link_reference}">
+      <sensor type="imu" name="${sensor_name}">
+        <always_on>true</always_on>
+        <update_rate>${update_rate}</update_rate>
+        <plugin filename="libgazebo_ros_imu_sensor.so" name="${sensor_name}_plugin">
+          <ros>
+            <namespace>/sensors</namespace>
+            <remapping>~/out:=imu/${topic_suffix}</remapping>
+          </ros>
+          <frame_name>${link_reference}</frame_name>
+          <static_reference>true</static_reference>
+          <gravity>true</gravity>
+          <orientation_reference_frame>ENU</orientation_reference_frame>
+        </plugin>
+        <imu>
+          <noise>
+            <type>gaussian</type>
+            <rate>
+              <mean>0.0</mean>
+              <stddev>0.0002</stddev>
+            </rate>
+            <accel>
+              <mean>0.0</mean>
+              <stddev>0.017</stddev>
+            </accel>
+          </noise>
+        </imu>
+      </sensor>
+    </gazebo>
+  </xacro:macro>
+  <!-- Transmission Macro -->
+  <xacro:macro name="joint_transmission" params="transmission_name joint_name actuator_name">
+    <transmission name="${transmission_name}">
+      <type>transmission_interface/SimpleTransmission</type>
+      <joint name="${joint_name}">
+        <hardwareInterface>hardware_interface/EffortJointInterface</hardwareInterface>
+      </joint>
+      <actuator name="${actuator_name}">
+        <mechanicalReduction>1</mechanicalReduction>
+        <hardwareInterface>hardware_interface/EffortJointInterface</hardwareInterface>
+      </actuator>
+    </transmission>
+  </xacro:macro>
+  <!-- Torque Sensor Macro -->
+  <xacro:macro name="torque_sensor"
+            params="reference_link
+                   sensor_name
+                   topic_suffix
+                   joint_name
+                   update_rate:=250
+                   frame:=child
+                   measure_direction:=child_to_parent
+                   force_stddev:=0.15
+                   torque_stddev:=0.02">
+    <gazebo reference="${reference_link}">
+      <sensor name="${sensor_name}" type="force_torque">
+        <update_rate>${update_rate}</update_rate>
+        <plugin filename="libgazebo_ros_ft_sensor.so" name="${sensor_name}_plugin">
+          <ros>
+            <namespace>/sensors</namespace>
+            <remapping>~/out:=joint_forces/${topic_suffix}</remapping>
+          </ros>
+          <joint_name>${joint_name}</joint_name>
+          <update_rate>${update_rate}</update_rate>
+          <frame_name>${joint_name}</frame_name>
+        </plugin>
+        <force_torque>
+          <frame>${frame}</frame>
+          <measure_direction>${measure_direction}</measure_direction>
+          <noise>
+            <type>gaussian</type>
+            <force>
+              <mean>0.0</mean>
+              <stddev>${force_stddev}</stddev>
+            </force>
+            <torque>
+              <mean>0.0</mean>
+              <stddev>${torque_stddev}</stddev>
+            </torque>
+          </noise>
+        </force_torque>
+      </sensor>
+    </gazebo>
+  </xacro:macro>
+<!-- Robot Definition -->
   <!-- Base Link with Motor Mass -->
   <link name="base_link">
     <inertial>
-      <origin xyz="0 0 0" rpy="0 0 0"/>
+      <origin xyz="0 0 1" rpy="0 0 0"/>
       <mass value="4.0"/>  <!-- 1.0kg base + 3.0kg motor -->
       <!-- Empirical inertia for 3kg motor (scaled from original) -->
@@ -37,6 +124,6 @@
     <!-- Positioned 2.5cm below base center-->
     <origin xyz="0 0 -0.025" rpy="0 0 0"/>
-    <!-- Z-axis rotation for flexion/extension -->
-    <axis xyz="0 0 1"/>
+    <!-- y-axis rotation for flexion/extension -->
+    <axis xyz="0 1 0"/>
     <!-- Limits for ISO 13485 Compliance -->
     <limit
@@ -59,104 +146,127 @@
     />
   </joint>
-<!-- Increased viscous damping --> <!-- Higher static friction -->
-<!-- Thigh Link with 3kg Motor Mass -->
-<link name="thigh_link">
-  <visual>
-    <geometry><cylinder length="0.3" radius="0.03"/></geometry>
-    <origin xyz="0 0 -0.15" rpy="0 0 0"/>
-    <material name="blue"><color rgba="0 0 0.8 1"/></material>
-  </visual>
-  <collision>
-    <geometry><cylinder length="0.3" radius="0.03"/></geometry>
-    <origin xyz="0 0 -0.15" rpy="0 0 0"/>
-  </collision>
-  <!-- Optimized Inertial for 3.5kg Total Mass -->
-  <inertial>
-    <origin xyz="0 0 0.2786"/>  <!-- COM: (0.5*0.15 + 3*0.3)/3.5 -->
-    <mass value="3.5"/>
-    <inertia
-      ixx="0.1135" ixy="0" ixz="0"
-      iyy="0.1135" iyz="0"
-      izz="0.000225"/>  <!-- Dominated by axial motor inertia -->
-  </inertial>
-</link>
-<gazebo reference="thigh_link">
-  <mu1>0.8</mu1>  <!-- Increased friction for heavy load -->
-  <mu2>0.8</mu2>
-  <kp>2000000</kp>  <!-- Higher stiffness -->
-  <kd>2000</kd>    <!-- Increased damping -->
-</gazebo>
-<!-- Optimized Knee Joint -->
-<joint name="knee_joint" type="revolute">
-  <parent link="thigh_link"/>
-  <child link="shank_link"/>
-  <!-- Corrected Origin (0.3m from parent origin) -->
-  <origin xyz="0 0 -0.3" rpy="0 0 0"/>  <!-- End of 0.3m thigh cylinder -->
-  <!-- Mediolateral Rotation Axis (Y-axis for sagittal plane motion) -->
-  <axis xyz="0 1 0"/>
-  <!-- Enhanced Dynamics for 3kg Motor -->
-  <dynamics damping="1.2" friction="0.4"/>  <!-- 8x higher damping than before -->
-  <!-- ISO 13485 Compliant Limits -->
-  <!-- 150° = 2.618 rad -->
-  <limit effort="350"
-         velocity="2.0"
-         lower="0"
-         upper="2.3"/>
-  <!-- Stronger braking force -->
-  <!-- 5.7° buffer for low limit-->
-  <!-- 6.8° buffer for upper limit-->
-  <safety_controller
-    k_velocity="150"
-    soft_lower_limit="0.05"
-    soft_upper_limit="2.2"/>
-</joint>
-<!-- Shank Link -->
-<link name="shank_link">
-  <visual>
-    <geometry><cylinder length="0.35" radius="0.025"/></geometry>
-    <origin xyz="0 0 -0.175" rpy="0 0 0"/>
-    <material name="red"><color rgba="0.8 0 0 1"/></material>
-  </visual>
-  <collision><geometry><cylinder length="0.35" radius="0.025"/></geometry></collision>
-  <inertial>
-    <mass value="0.3"/>
-    <inertia ixx="0.003" ixy="0" ixz="0" iyy="0.003" iyz="0" izz="0.003"/>
-  </inertial>
-  <!-- Gazebo Attr -->
+  <!-- Increased viscous damping --> <!-- Higher static friction -->
+  <!-- Thigh Link with 3kg Motor Mass -->
+  <link name="thigh_link">
+    <visual>
+      <geometry><cylinder length="0.3" radius="0.03"/></geometry>
+      <origin xyz="0 0 -0.15" rpy="0 0 0"/>
+      <material name="blue"><color rgba="0 0 0.8 1"/></material>
+    </visual>
+    <collision>
+      <geometry><cylinder length="0.3" radius="0.03"/></geometry>
+      <origin xyz="0 0 -0.15" rpy="0 0 0"/>
+    </collision>
+    <!-- Optimized Inertial for 3.5kg Total Mass -->
+    <inertial>
+      <origin xyz="0 0 0.2786"/>  <!-- COM: (0.5*0.15 + 3*0.3)/3.5 -->
+      <mass value="3.5"/>
+      <inertia
+        ixx="0.1135" ixy="0" ixz="0"
+        iyy="0.1135" iyz="0"
+        izz="0.000225"/>  <!-- Dominated by axial motor inertia -->
+    </inertial>
+  </link>
+  <gazebo reference="thigh_link">
+    <mu1>0.8</mu1>  <!-- Increased friction for heavy load -->
+    <mu2>0.8</mu2>
+    <kp>2000000</kp>  <!-- Higher stiffness -->
+    <kd>2000</kd>    <!-- Increased damping -->
+  </gazebo>
+  <!-- Knee Joint -->
+  <joint name="knee_joint" type="revolute">
+    <parent link="thigh_link"/>
+    <child link="shank_link"/>
+    <!-- Corrected Origin (0.3m from parent origin) -->
+    <origin xyz="0 0 -0.3" rpy="0 0 0"/>  <!-- End of 0.3m thigh cylinder -->
+    <!-- Mediolateral Rotation Axis (Y-axis for sagittal plane motion) -->
+    <axis xyz="0 1 0"/>
+    <!-- Enhanced Dynamics for 3kg Motor -->
+    <dynamics damping="1.2" friction="0.4"/>  <!-- 8x higher damping than before -->
+    <!-- ISO 13485 Compliant Limits -->
+    <!-- 150° = 2.618 rad -->
+    <limit effort="350"
+          velocity="2.0"
+          lower="0"
+          upper="2"/>
+    <!-- Stronger braking force -->
+    <!-- 5.7° buffer for low limit-->
+    <!-- 6.8° buffer for upper limit-->
+    <safety_controller
+      k_velocity="150"
+      soft_lower_limit="0.05"
+      soft_upper_limit="1.9"/>
+  </joint>
+  <!-- Shank Link -->
+  <link name="shank_link">
+    <visual>
+      <geometry>
+        <cylinder length="0.35" radius="0.025"/>
+      </geometry>
+      <!-- Center cylinder at link origin -->
+      <origin xyz="0 0 -0.175" rpy="0 0 0"/>
+      <material name="red">
+        <color rgba="0.8 0 0 1"/>
+      </material>
+    </visual>
+    <collision>
+      <geometry>
+        <cylinder length="0.35" radius="0.025"/>
+      </geometry>
+      <!-- Match visual origin -->
+      <origin xyz="0 0 0" rpy="0 0 0"/>
+    </collision>
+    <!-- Optimized Inertial Properties -->
+    <inertial>
+      <origin xyz="0 0 0.175"/>  <!-- COM at geometric center -->
+      <mass value="0.25"/>  <!-- Increased from 0.3kg for safety margin -->
+      <!--
+        Cylinder inertia formulas (r=0.025m, h=0.35m):
+        I_xx = I_yy = (1/12)*m*(3r² + h²) = 0.00257
+        I_zz = (1/2)*m*r² = 0.000078
+      -->
+      <inertia
+        ixx="0.00257" ixy="0" ixz="0"
+        iyy="0.00257" iyz="0"
+        izz="0.000078"/>
+    </inertial>
+  </link>
+  <!-- Shank Link Gazebo Attr -->
   <gazebo reference="shank_link">
-    <mu1>0.2</mu1>  <!-- Contact Friction Coefficient -->
-    <mu2>0.2</mu2>
-    <kp>1000000</kp>  <!-- Contact Stiffness [N/m] -->
-    <kd>100</kd>      <!-- Contact Damping [N·s/m] -->
-  </gazebo>
-</link>
-<!-- Ankle Joint -->
-<joint name="ankle_joint" type="revolute">
-  <parent link="shank_link"/>
-  <child link="foot_link"/>
-  <!-- Position ankle joint at the end of shank_link -->
-  <origin xyz="0 0 -0.35" rpy="0 0 0"/> <!-- Negative Z to move down from shank_link -->
-  <axis xyz="0 1 0"/>
-  <dynamics damping="0.03" friction="0.005"/>
-  <!--
-    typical ROM for ankle joint is 20° dorsiflexion and 50° plantarflexion
-    Dorsiflexion (upward movement)‌: 0 - 20° (0 - 0.35rad)
-    Plantarflexion (downward movement)‌: 0 - 55° (0 - 0.96rad)
-  -->
-  <limit effort="300" velocity="3.0" lower="-0.3" upper="0.3"/>
-  <safety_controller k_velocity="50" soft_lower_limit="-0.25" soft_upper_limit="0.25"/>
-</joint>
-<!-- Foot Link -->
-<link name="foot_link">
-  <visual>
-    <geometry><box size="0.15 0.05 0.01"/></geometry>
-    <material name="gray"><color rgba="0.5 0.5 0.5 1"/></material>
-  </visual>
-  <collision><geometry><box size="0.15 0.05 0.01"/></geometry></collision>
-  <inertial>
-    <mass value="0.1"/>
-    <inertia ixx="0.0001" ixy="0" ixz="0" iyy="0.0001" iyz="0" izz="0.0001"/>
-  </inertial>
-  <!-- Gazebo Attr -->
+    <material>Gazebo/Red</material>
+    <mu1>0.6</mu1>  <!-- Increased friction for fabric grip -->
+    <mu2>0.6</mu2>
+    <kp>50000</kp>   <!-- Reduced stiffness for stability -->
+    <kd>500</kd>     <!-- Increased damping -->
+  </gazebo>
+  <!-- Ankle Joint -->
+  <joint name="ankle_joint" type="revolute">
+    <parent link="shank_link"/>
+    <child link="foot_link"/>
+    <!-- Position ankle joint at the end of shank_link -->
+    <origin xyz="0.015 0 -0.36" rpy="0 0 0"/> <!-- Negative Z to move down from shank_link -->
+    <axis xyz="0 1 0"/>
+    <dynamics damping="0.8" friction="0.1"/>
+    <!--
+      typical ROM for ankle joint is 20° dorsiflexion and 50° plantarflexion
+      Dorsiflexion (upward movement)‌: 0 - 20° (0 - 0.35rad)
+      Plantarflexion (downward movement)‌: 0 - 55° (0 - 0.96rad)
+    -->
+    <limit effort="150" velocity="3.0" lower="-0.3" upper="0.3"/>
+    <safety_controller k_velocity="100" soft_lower_limit="-0.25" soft_upper_limit="0.25"/>
+  </joint>
+  <!-- Foot Link -->
+  <link name="foot_link">
+    <visual>
+      <geometry><box size="0.18 0.07 0.04"/></geometry>
+      <material name="gray"><color rgba="0.5 0.5 0.5 1"/></material>
+    </visual>
+    <collision><geometry><box size="0.15 0.05 0.01"/></geometry></collision>
+    <inertial>
+      <mass value="0.1"/>
+      <inertia ixx="0.0001" ixy="0" ixz="0" iyy="0.0001" iyz="0" izz="0.0001"/>
+    </inertial>
+  </link>
+  <!-- Foot Link Gazebo Attr -->
   <gazebo reference="foot_link">
     <mu1>0.2</mu1>  <!-- Contact Friction Coefficient -->
@@ -165,110 +275,56 @@
     <kd>100</kd>      <!-- Contact Damping [N·s/m] -->
   </gazebo>
-</link>
-<!-- Transmissions -->
-<transmission name="hip_transmission">
-  <type>transmission_interface/SimpleTransmission</type>
-  <actuator name="hip_motor">
-    <hardwareInterface>Effort</hardwareInterface>
-  </actuator>
-  <joint name="hip_joint"/>
-</transmission>
-<transmission name="knee_transmission">
-  <type>transmission_interface/SimpleTransmission</type>
-  <actuator name="knee_motor">
-    <hardwareInterface>Effort</hardwareInterface>
-  </actuator>
-  <joint name="knee_joint"/>
-</transmission>
-<transmission name="ankle_transmission">
-  <type>transmission_interface/SimpleTransmission</type>
-  <actuator name="ankle_motor">
-    <hardwareInterface>Effort</hardwareInterface>
-  </actuator>
-  <joint name="ankle_joint"/>
-</transmission>
+<!-- Gazebo Transmissions -->
+  <!-- Corrected Transmissions -->
+  <xacro:joint_transmission
+      transmission_name="hip_transmission"
+      joint_name="hip_joint"
+      actuator_name="hip_motor"
+  />
+  <xacro:joint_transmission
+      transmission_name="knee_transmission"
+      joint_name="knee_joint"
+      actuator_name="knee_motor"
+  />
+  <xacro:joint_transmission
+      transmission_name="ankle_transmission"
+      joint_name="ankle_joint"
+      actuator_name="ankle_motor"
+  />
 <!-- Gazebo Sensor Plugin -->
-<!-- IMU -->
-<gazebo reference="thigh_link">
-  <sensor type="imu" name="thigh_link">
-    <always_on>true</always_on>
-    <update_rate>100</update_rate>
-    <plugin filename="libgazebo_ros_imu_sensor.so" name="imu_plugin">
-      <ros>
-        <namespace>/</namespace>
-        <remapping>~/out:=/imu/thigh_link_data</remapping>  <!-- custom topic name -->
-      </ros>
-      <frame_name>thigh_link</frame_name>  <!-- must be the same with reference -->
-    </plugin>
-  </sensor>
-</gazebo>
-<gazebo reference="foot_link">
-  <sensor type="imu" name="foot_imu">
-    <always_on>true</always_on>
-    <update_rate>100</update_rate>
-    <plugin filename="libgazebo_ros_imu_sensor.so" name="imu_plugin">
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
Commit message: fixed gazebo plugins for sensors

File: src/exo_urdf/urdf/exo.urdf (robot description, URDF)
Before this commit: robot exo_urdf, 4 links, 3 joints
Links:
- added link world
- link foot_link: geometry collision box size=0.15 0.05 0.01; visual box size=0.18 0.07 0.04
Joints:
- added joint fixed_joint: type fixed, parent world, child base_link, origin xyz=0 0 1 rpy=0 0 0
- joint ankle_joint: origin xyz=0 0 -0.35 rpy=0 0 0 -> xyz=0.015 0 -0.36 rpy=0 0 0
- joint hip_joint: axis 0 0 1 -> 0 1 0
- joint knee_joint: limit lower=0 upper=2.3 effort=350 velocity=2.0 -> lower=0 upper=2 effort=350 velocity=2.0

File: src/exo_urdf/urdf/exo.xacro (robot description, xacro)
@@ -4,4 +4,17 @@
   <xacro:property name="motor_mass" value="3" />  <!-- Hip / Knee motor mass (kg) -->
   <xacro:property name="base_mass" value="1.0" />   <!-- Base structure mass -->
+  <!-- Transmission Macro -->
+  <xacro:macro name="joint_transmission" params="transmission_name joint_name actuator_name">
+    <transmission name="${transmission_name}">
+      <type>transmission_interface/SimpleTransmission</type>
+      <joint name="${joint_name}">
+        <hardwareInterface>hardware_interface/EffortJointInterface</hardwareInterface>
+      </joint>
+      <actuator name="${actuator_name}">
+        <mechanicalReduction>1</mechanicalReduction>
+        <hardwareInterface>hardware_interface/EffortJointInterface</hardwareInterface>
+      </actuator>
+    </transmission>
+  </xacro:macro>
   <!-- IMU Sensor Macro -->
   <xacro:macro name="imu_sensor" params="link_reference sensor_name topic_suffix update_rate:=100">
@@ -36,63 +49,41 @@
     </gazebo>
   </xacro:macro>
-  <!-- Transmission Macro -->
-  <xacro:macro name="joint_transmission" params="transmission_name joint_name actuator_name">
-    <transmission name="${transmission_name}">
-      <type>transmission_interface/SimpleTransmission</type>
-      <joint name="${joint_name}">
-        <hardwareInterface>hardware_interface/EffortJointInterface</hardwareInterface>
-      </joint>
-      <actuator name="${actuator_name}">
-        <mechanicalReduction>1</mechanicalReduction>
-        <hardwareInterface>hardware_interface/EffortJointInterface</hardwareInterface>
-      </actuator>
-    </transmission>
-  </xacro:macro>
-  <!-- Torque Sensor Macro -->
-  <xacro:macro name="torque_sensor"
-            params="reference_link
-                   sensor_name
-                   topic_suffix
-                   joint_name
-                   update_rate:=250
-                   frame:=child
-                   measure_direction:=child_to_parent
-                   force_stddev:=0.15
-                   torque_stddev:=0.02">
-    <gazebo reference="${reference_link}">
-      <sensor name="${sensor_name}" type="force_torque">
-        <update_rate>${update_rate}</update_rate>
-        <plugin filename="libgazebo_ros_ft_sensor.so" name="${sensor_name}_plugin">
-          <ros>
-            <namespace>/sensors</namespace>
-            <remapping>~/out:=joint_forces/${topic_suffix}</remapping>
-          </ros>
-          <joint_name>${joint_name}</joint_name>
-          <update_rate>${update_rate}</update_rate>
-          <frame_name>${joint_name}</frame_name>
-        </plugin>
-        <force_torque>
-          <frame>${frame}</frame>
-          <measure_direction>${measure_direction}</measure_direction>
-          <noise>
-            <type>gaussian</type>
-            <force>
-              <mean>0.0</mean>
-              <stddev>${force_stddev}</stddev>
-            </force>
-            <torque>
-              <mean>0.0</mean>
-              <stddev>${torque_stddev}</stddev>
-            </torque>
-          </noise>
-        </force_torque>
-      </sensor>
-    </gazebo>
-  </xacro:macro>
+  <!-- Macro Definition (Revised) -->
+  <xacro:macro name="torque_sensor" params="reference_link sensor_name topic_suffix joint_name force_stddev torque_stddev">
+  <!-- Enable feedback on the joint (critical for FT sensors) -->
+  <gazebo reference="${joint_name}">
+    <provideFeedback>true</provideFeedback>
+  </gazebo>
+  <!-- Sensor definition -->
+  <gazebo>
+    <plugin name="${sensor_name}_plugin" filename="libgazebo_ros_ft_sensor.so">
+      <update_rate>1000</update_rate>
+      <ros>
+        <namespace>/sensors/torque/${topic_suffix}</namespace>
+      </ros>
+      <joint_name>${joint_name}</joint_name>
+      <noise>
+        <force>
+          <stddev>${force_stddev}</stddev>
+        </force>
+        <torque>
+          <stddev>${torque_stddev}</stddev>
+        </torque>
+      </noise>
+    </plugin>
+  </gazebo>
+</xacro:macro>
 <!-- Robot Definition -->
+  <link name="world"/>  <!-- Dummy link for Gazebo's world frame -->
+    <!-- Optional: Add a world-fixed joint -->
+    <joint name="fixed_joint" type="fixed">
+      <parent link="world"/>
+      <child link="base_link"/>
+      <origin xyz="0 0 1" rpy="0 0 0"/>  <!-- 1m above ground -->
+  </joint>
   <!-- Base Link with Motor Mass -->
   <link name="base_link">
     <inertial>
-      <origin xyz="0 0 1" rpy="0 0 0"/>
+      <origin xyz="0 0 0" rpy="0 0 0"/>
       <mass value="4.0"/>  <!-- 1.0kg base + 3.0kg motor -->
       <!-- Empirical inertia for 3kg motor (scaled from original) -->
@@ -296,34 +287,43 @@
   <xacro:imu_sensor link_reference="thigh_link"
                   sensor_name="thigh_imu_sensor"
-                  topic_suffix="thigh"/>
+                  topic_suffix="thigh"
+  />
   <!-- Shank IMU -->
   <xacro:imu_sensor link_reference="shank_link"
                   sensor_name="shank_imu_sensor"
-                  topic_suffix="shank"/>
+                  topic_suffix="shank"
+  />
   <!-- Foot IMU -->
   <xacro:imu_sensor link_reference="foot_link"
                   sensor_name="foot_imu_sensor"
-                  topic_suffix="foot"/>
+                  topic_suffix="foot"
+  />
 <!-- Gazebo Torque Sensors Plugin -->
-<!-- Hip Torque -->
-<xacro:torque_sensor
+  <!-- Hip Torque -->
+  <xacro:torque_sensor
     reference_link="thigh_link"
     sensor_name="hip_torque_sensor"
     topic_suffix="hip"
     joint_name="hip_joint"
-/>
-<!-- Knee Torque -->
-<xacro:torque_sensor
+    force_stddev="0.15"
+    torque_stddev="0.02"
+  />
+  <!-- Knee Torque -->
+  <xacro:torque_sensor
     reference_link="shank_link"
     sensor_name="knee_torque_sensor"
     topic_suffix="knee"
     joint_name="knee_joint"
-/>
+    force_stddev="0.15"
+    torque_stddev="0.02"
+  />
 <!-- Ankle Torque -->
 <xacro:torque_sensor
-    reference_link="foot_link"
-    sensor_name="ankle_torque_sensor"
-    topic_suffix="ankle"
-    joint_name="ankle_joint"
+  reference_link="foot_link"
+  sensor_name="ankle_torque_sensor"
+  topic_suffix="ankle"
+  joint_name="ankle_joint"
+  force_stddev="0.15"
+  torque_stddev="0.02"
 />
   <!-- Contact Sensor -->
