Commit message: separated the URDF into multiple files

File: src/exo_urdf/urdf/exo.urdf.xacro (robot description, xacro)
@@ -1,6 +1,18 @@
 <?xml version="1.0"?>
 <robot name="exo" xmlns:xacro="http://ros.org/wiki/xacro">
+<!-- Properties -->
+<xacro:property name="motor_mass" value="3" />  <!-- Hip / Knee motor mass (kg) -->
+<xacro:property name="base_mass" value="1.0" />   <!-- Base structure mass -->
+<!-- Macros -->
+<xacro:include filename="$(find exo_urdf)/urdf/transmission_macro.xacro" />
+<xacro:include filename="$(find exo_urdf)/urdf/sensor_IMU_macro.xacro" />
+<xacro:include filename="$(find exo_urdf)/urdf/sensor_torque_macro.xacro" />
+<!-- Robot Description (link / joint) -->
 <xacro:include filename="$(find exo_urdf)/urdf/robot_description.xacro" />
+<!-- Gazebo Transmission -->
 <xacro:include filename="$(find exo_urdf)/urdf/transmission.xacro" />
+<!-- Sensors -->
+<xacro:include filename="$(find exo_urdf)/urdf/sensor.xacro" />
+<!-- ROS2 Control -->
 <xacro:include filename="$(find exo_urdf)/urdf/ros2_control.xacro" />
 </robot>

File: src/exo_urdf/urdf/robot_description.xacro (robot description, xacro)
@@ -1,7 +1,4 @@
 <?xml version="1.0"?>
 <robot xmlns:xacro="http://www.ros.org/wiki/xacro">
-<!-- Properties -->
-  <xacro:property name="motor_mass" value="3.0" />  <!-- Hip / Knee motor mass (kg) -->
-  <xacro:property name="base_mass" value="1.0" />   <!-- Base structure mass -->
 <!-- Robot Definition -->
   <link name="world"/>  <!-- Dummy link for Gazebo's world frame -->
@@ -16,5 +13,5 @@
     <inertial>
       <origin xyz="0 0 0" rpy="0 0 0"/>
-      <mass value="motor_mass + base_mass"/>  <!-- 1.0kg base + 3.0kg motor -->
+      <mass value="4.0"/>  <!-- 1.0kg base + 3.0kg motor -->
       <!-- Empirical inertia for 3kg motor (scaled from original) -->
       <inertia

File: src/exo_urdf/urdf/ros2_control.xacro (robot description, xacro)
@@ -2,18 +2,19 @@
 <robot xmlns:xacro="http://www.ros.org/wiki/xacro">
 <!-- ROS Control Configuration -->
-  <ros2_control name="exo_hardware" type="system">
+  <ros2_control name="exo" type="system">
     <hardware>
       <plugin>gazebo_ros2_control/GazeboSystem</plugin>
     </hardware>
+    <!-- Define all 3 joints here -->
     <joint name="hip_joint">
-      <command_interface name="position"/>  <!-- Position control for PID -->
+      <command_interface name="effort"/>  <!-- Effort control for PID -->
       <state_interface name="position"/>  <!-- Feedback from the joint -->
     </joint>
     <joint name="knee_joint">
-      <command_interface name="position"/>
+      <command_interface name="effort"/>
       <state_interface name="position"/>
     </joint>
     <joint name="ankle_joint">
-      <command_interface name="position"/>
+      <command_interface name="effort"/>
       <state_interface name="position"/>
     </joint>
@@ -25,4 +26,5 @@
       <controlPeriod>0.001</controlPeriod>  <!-- 1kHz control rate -->
       <robotParam>robot_description</robotParam>
+      <parameters>$(find exo_urdf)/config/controllers.yaml</parameters>
     </plugin>
   </gazebo>

File: src/exo_urdf/urdf/sensor.xacro (robot description, xacro)
@@ -1,6 +1,4 @@
 <?xml version="1.0"?>
 <robot xmlns:xacro="http://www.ros.org/wiki/xacro">
-<xacro:include filename="$(find exo_urdf)/urdf/sensor_IMU_macro.xacro" />
-<xacro:include filename="$(find exo_urdf)/urdf/sensor_torque_macro.xacro" />
 <!-- Gazebo IMU Sensor Plugin -->
   <!-- Thigh IMU -->
@@ -54,16 +52,3 @@
     </sensor>
   </gazebo>
-  <gazebo>
-    <plugin name="exo_ros_control" filename="libgazebo_ros_control.so">
-      <robotNamespace>/exo</robotNamespace>
-      <controlPeriod>0.001</controlPeriod>  <!-- 1kHz control rate -->
-      <robotParam>robot_description</robotParam>
-    </plugin>
-  </gazebo>
-  <gazebo>
-    <physics type="ode">
-      <max_step_size>0.002</max_step_size>
-      <real_time_update_rate>500</real_time_update_rate>
-    </physics>
-  </gazebo>
 </robot>

File: src/exo_urdf/urdf/sensor_IMU_macro.xacro (robot description, xacro)
@@ -1,5 +1,5 @@
 <?xml version="1.0"?>
 <robot xmlns:xacro="http://www.ros.org/wiki/xacro">
-<!-- IMU Sensor Macro -->
+  <!-- IMU Sensor Macro -->
   <xacro:macro name="imu_sensor" params="link_reference sensor_name topic_suffix update_rate:=100">
     <gazebo reference="${link_reference}">

File: src/exo_urdf/urdf/transmission.xacro (robot description, xacro)
@@ -1,5 +1,4 @@
 <?xml version="1.0"?>
 <robot xmlns:xacro="http://www.ros.org/wiki/xacro">
-<xacro:include filename="$(find exo_urdf)/urdf/transmission_macro.xacro" />
 <!-- Gazebo Transmissions -->
   <!-- Corrected Transmissions -->

File: src/exo_urdf/urdf/transmission_macro.xacro (robot description, xacro)
@@ -1,5 +1,5 @@
 <?xml version="1.0"?>
 <robot xmlns:xacro="http://www.ros.org/wiki/xacro">
-<!-- Transmission Macro -->
+  <!-- Transmission Macro -->
   <xacro:macro name="joint_transmission" params="transmission_name joint_name actuator_name hardware_interface:=EffortJointInterface mechanical_reduction:=1">
     <transmission name="${transmission_name}">
